Commit message: Imported upstream version '1.3.0' of 'upstream'

File: nav2_minimal_tb3_sim/urdf/gz_waffle_gps.sdf.xacro (robot description, xacro)
@@ -44,5 +44,5 @@
           <update_rate>200</update_rate>
           <topic>$(arg namespace)/imu/data</topic>
-          <gz_frame_id>imu_link</gz_frame_id>
+          <frame_id>imu_link</frame_id>
           <imu>
             <angular_velocity>
@@ -94,8 +94,10 @@
           <update_rate>1</update_rate>
           <topic>$(arg namespace)/gps/fix</topic>
-          <gz_frame_id>gps_link</gz_frame_id>
+          <frame_id>gps_link</frame_id>
           <navsat>
             <position_sensing>
               <horizontal>
+              <!-- Be carefull setting this.
+              Units in degree not in meters https://github.com/gazebosim/sdformat/issues/1572 -->
                 <noise type="gaussian">
                   <mean>0.0</mean>
@@ -144,5 +146,5 @@
           </geometry>
           <material>
-            <diffuse>1 1 1</diffuse>
+            <diffuse>0.5 0.5 0.5</diffuse>
           </material>
         </visual>
@@ -153,5 +155,5 @@
           <update_rate>5</update_rate>
           <topic>$(arg namespace)/scan</topic>
-          <gz_frame_id>base_scan</gz_frame_id>
+          <frame_id>base_scan</frame_id>
           <ray>
             <scan>
@@ -199,5 +201,5 @@
           <surface>
             <friction>
-              <ode>
+              <bullet>
                 <mu>1</mu>
                 <mu2>1</mu2>
@@ -205,8 +207,8 @@
                 <slip2>0</slip2>
                 <fdir1>0 0 1</fdir1>
-              </ode>
+              </bullet>
             </friction>
             <contact>
-              <ode>
+              <bullet>
                 <soft_cfm>0</soft_cfm>
                 <soft_erp>0.2</soft_erp>
@@ -215,5 +217,5 @@
                 <max_vel>0.01</max_vel>
                 <min_depth>0.001</min_depth>
-              </ode>
+              </bullet>
             </contact>
           </surface>
@@ -228,5 +230,5 @@
           </geometry>
           <material>
-            <diffuse>1 1 1</diffuse>
+            <diffuse>0.5 0.5 0.5</diffuse>
           </material>
         </visual>
@@ -255,5 +257,5 @@
           <surface>
             <friction>
-              <ode>
+              <bullet>
                 <mu>1</mu>
                 <mu2>1</mu2>
@@ -261,8 +263,8 @@
                 <slip2>0</slip2>
                 <fdir1>0 0 1</fdir1>
-              </ode>
+              </bullet>
             </friction>
             <contact>
-              <ode>
+              <bullet>
                 <soft_cfm>0</soft_cfm>
                 <soft_erp>0.2</soft_erp>
@@ -271,5 +273,5 @@
                 <max_vel>0.01</max_vel>
                 <min_depth>0.001</min_depth>
-              </ode>
+              </bullet>
             </contact>
           </surface>
@@ -284,10 +286,10 @@
           </geometry>
           <material>
-            <diffuse>1 1 1</diffuse>
+            <diffuse>0.5 0.5 0.5</diffuse>
           </material>
         </visual>
       </link>
       <link name='caster_back_right_link'>
-        <pose>-0.177 -0.064 -0.004 0 0 0</pose>
+        <pose>-0.177 -0.064 -0.004 -1.57 0 0</pose>
         <inertial>
           <mass>0.001</mass>
@@ -301,13 +303,13 @@
           </inertia>
         </inertial>
-        <collision name='collision'>
+        <collision name='caster_back_right_collision'>
           <geometry>
             <sphere>
-              <radius>0.005000</radius>
+              <radius>0.0060000</radius>
             </sphere>
           </geometry>
           <surface>
             <contact>
-              <ode>
+              <bullet>
                 <soft_cfm>0</soft_cfm>
                 <soft_erp>0.2</soft_erp>
@@ -316,11 +318,21 @@
                 <max_vel>0.01</max_vel>
                 <min_depth>0.001</min_depth>
-              </ode>
+              </bullet>
             </contact>
           </surface>
         </collision>
+        <visual name="sphere_visual">
+          <geometry>
+            <sphere>
+              <radius>0.0060000</radius>
+            </sphere>
+          </geometry>
+          <material>
+            <diffuse>0.5 0.5 0.5</diffuse>
+          </material>
+        </visual>
       </link>
       <link name='caster_back_left_link'>
-        <pose>-0.177 0.064 -0.004 0 0 0</pose>
+        <pose>-0.177 0.064 -0.004 -1.57 0 0</pose>
         <inertial>
           <mass>0.001</mass>
@@ -334,13 +346,13 @@
           </inertia>
         </inertial>
-        <collision name='collision'>
+        <collision name='caster_back_left_collision'>
           <geometry>
             <sphere>
-              <radius>0.005000</radius>
+              <radius>0.0060000</radius>
             </sphere>
           </geometry>
           <surface>
             <contact>
-              <ode>
+              <bullet>
                 <soft_cfm>0</soft_cfm>
                 <soft_erp>0.2</soft_erp>
@@ -349,8 +361,18 @@
                 <max_vel>0.01</max_vel>
                 <min_depth>0.001</min_depth>
-              </ode>
+              </bullet>
             </contact>
           </surface>
         </collision>
+       <visual name="sphere_visual">
+          <geometry>
+            <sphere>
+              <radius>0.0060000</radius>
+            </sphere>
+          </geometry>
+          <material>
+            <diffuse>0.5 0.5 0.5</diffuse>
+          </material>
+        </visual>
       </link>
       <link name="camera_link">
@@ -380,5 +402,5 @@
           <update_rate>5</update_rate>
           <pose>0.064 -0.047 0.107 0 0 0</pose>
-          <gz_frame_id>camera_depth_frame</gz_frame_id>
+          <frame_id>camera_depth_frame</frame_id>
           <camera name="realsense_depth_camera">
             <horizontal_fov>1.047</horizontal_fov>
@@ -461,8 +483,10 @@
         filename="gz-sim-diff-drive-system"
         name="gz::sim::systems::DiffDrive">
+        <!-- wheel information -->
         <left_joint>wheel_left_joint</left_joint>
         <right_joint>wheel_right_joint</right_joint>
         <wheel_separation>0.287</wheel_separation>
         <wheel_radius>0.033</wheel_radius>
+        <!-- limits -->
         <max_linear_acceleration>1</max_linear_acceleration>
         <min_linear_acceleration>-1</min_linear_acceleration>
@@ -473,5 +497,7 @@
         <max_angular_velocity>1.9</max_angular_velocity>
         <min_angular_velocity>-1.9</min_angular_velocity>
+        <!-- input -->
         <topic>$(arg namespace)/cmd_vel</topic>
+        <!-- output -->
         <odom_topic>$(arg namespace)/odom</odom_topic>
         <tf_topic>$(arg namespace)/tf</tf_topic>
